Commit message: Fixed Comments

File: ecm_description/urdf/xacros/ecm.xacro (robot description, xacro)
@@ -159,9 +159,7 @@
             <child link="${prefix}_yaw_link" />
             <origin rpy="0 -${PI/2} ${PI/2}" xyz="0 0 0" />
-            <!--rotates
-            about z axis-->
-            <axis xyz="0 0 1" />
-            <!--limit
-            effort and velocity picked arbitrarily check-->
+            <!-- Rotates about z axis -->
+            <axis xyz="0 0 1" />
+            <!-- Limit effort and velocity picked arbitrarily check -->
             <limit effort="50.0" lower="${-75/180*PI}" upper="${PI/4}" velocity="2" />
             <joint_properties damping="1.0" friction="0.0" />

File: mtm_description/urdf/xacros/mtm.xacro (robot description, xacro)
@@ -125,9 +125,7 @@
             <child link="${prefix}_outer_yaw_link" />
             <origin rpy="0 0 ${PI/2}" xyz="0 0 0" />
-            <!--rotates
-            about z axis-->
-            <axis xyz="0 0 1" />
-            <!--limit
-            effort and velocity picked arbitrarily check-->
+            <!-- Rotates about z axis -->
+            <axis xyz="0 0 1" />
+            <!-- Limit effort and velocity picked arbitrarily check -->
             <limit effort="50.0" lower="${-75/180*PI}" upper="${PI/4}" velocity="2" />
             <joint_properties damping="1.0" friction="0.0" />
@@ -139,6 +137,5 @@
             <origin rpy="${-PI/2} ${-PI/2} 0" xyz="0 0 0" />
             <axis xyz="0 0 1" />
-            <!--limit
-            effort and velocity picked arbitrarily check-->
+            <!-- Limit effort and velocity picked arbitrarily check -->
             <limit effort="100.0" lower="${-PI/4}" upper="${PI/4}" velocity="10" />
             <joint_properties damping="1.0" friction="0.0" />
@@ -149,9 +146,7 @@
             <child link="${prefix}_top_parallel_link" />
             <origin rpy="${-PI/2} ${-PI/2} 0" xyz="0 0 0" />
-            <!--rotates
-            about x axis-->
-            <axis xyz="0 0 1" />
-            <!--limit
-            effort and velocity picked arbitrarily check-->
+            <!-- Rotates about x axis -->
+            <axis xyz="0 0 1" />
+            <!-- Limit effort and velocity picked arbitrarily check -->
             <limit effort="100.0" lower="${-PI/2}" upper="${PI/2}" velocity="10" />
             <joint_properties damping="1.0" friction="0.0" />
@@ -164,6 +159,5 @@
             <origin rpy="0 0 ${PI/2}" xyz="-0.2794 0 0" />
             <axis xyz="0 0 1" />
-            <!--limit
-            effort and velocity picked arbitrarily check-->
+            <!-- Limit effort and velocity picked arbitrarily check -->
             <limit effort="100.0" lower="${-PI/4}" upper="${PI/4}" velocity="10" />
             <joint_properties damping="1.0" friction="0.0" />
@@ -287,9 +281,7 @@
             <child link="${prefix}_wrist_platform_link" />
             <origin rpy="${PI/2} 0 0" xyz="-0.3645 -0.1506 0.0" />
-            <!--rotates
-            about z axis-->
-            <axis xyz="0 0 1" />
-            <!--limit
-            effort and velocity picked arbitrarily check-->
+            <!-- Rotates about z axis -->
+            <axis xyz="0 0 1" />
+            <!-- Limit effort and velocity picked arbitrarily check -->
             <limit effort="100.0" lower="${-60/180*PI}" upper="${245/180*PI}" velocity="10" />
             <joint_properties damping="1.0" friction="0.0" />
@@ -301,6 +293,5 @@
             <origin rpy="${-PI/2} 0 0" xyz="0 0 0" />
             <axis xyz="0 0 1" />
-            <!--limit
-            effort and velocity picked arbitrarily check-->
+            <!-- Limit effort and velocity picked arbitrarily check -->
             <limit effort="100.0" lower="${-PI/2}" upper="${PI}" velocity="10" />
             <joint_properties damping="1.0" friction="0.0" />
@@ -311,9 +302,7 @@
             <child link="${prefix}_wrist_yaw_link" />    <!--  defined from CAD file-->
             <origin rpy="${PI/2} ${-PI/2} 0" xyz="0 0 0" />
-            <!--rotates
-            about z axis-->
-            <axis xyz="0 0 1" />
-            <!--limit
-            effort and velocity picked arbitrarily check-->
+            <!-- Rotates about z axis -->
+            <axis xyz="0 0 1" />
+            <!-- Limit effort and velocity picked arbitrarily check -->
             <limit effort="100.0" lower="${-PI/4}" upper="${PI/4}" velocity="10" />
             <joint_properties damping="1.0" friction="0.0" />
@@ -326,6 +315,5 @@
             <origin rpy="0 ${-PI/2} ${PI/2}" xyz="0 0 0" />
             <axis xyz="0 0 1" />
-            <!--limit
-            effort and velocity picked arbitrarily check-->
+            <!-- Limit effort and velocity picked arbitrarily check -->
             <limit effort="100.0" lower="${-1.5*PI}" upper="${1.5*PI}" velocity="10" />
             <joint_properties damping="1.0" friction="0.0" />
@@ -447,9 +435,7 @@
             <child link="${prefix}_wrist_platform_link" />
             <origin rpy="${PI/2} 0 0" xyz="-0.3645 -0.1506 0.0" />
-            <!--rotates
-            about z axis-->
-            <axis xyz="0 0 1" />
-            <!--limit
-            effort and velocity picked arbitrarily check-->
+            <!-- Rotates about z axis -->
+            <axis xyz="0 0 1" />
+            <!-- Limit effort and velocity picked arbitrarily check -->
             <limit effort="100.0" lower="${-60/180*PI}" upper="${245/180*PI}" velocity="10" />
             <joint_properties damping="1.0" friction="0.0" />
@@ -461,6 +447,5 @@
             <origin rpy="${-PI/2} 0 0" xyz="0 0 0" />
             <axis xyz="0 0 1" />
-            <!--limit
-            effort and velocity picked arbitrarily check-->
+            <!-- Limit effort and velocity picked arbitrarily check -->
             <limit effort="100.0" lower="${-PI/2}" upper="${PI}" velocity="10" />
             <joint_properties damping="1.0" friction="0.0" />
@@ -471,9 +456,7 @@
             <child link="${prefix}_wrist_yaw_link" />    <!--  defined from CAD file-->
             <origin rpy="${PI/2} ${-PI/2} 0" xyz="0 0 0" />
-            <!--rotates
-            about z axis-->
-            <axis xyz="0 0 1" />
-            <!--limit
-            effort and velocity picked arbitrarily check-->
+            <!-- Rotates about z axis -->
+            <axis xyz="0 0 1" />
+            <!-- Limit effort and velocity picked arbitrarily check -->
             <limit effort="100.0" lower="${-PI/4}" upper="${PI/4}" velocity="10" />
             <joint_properties damping="1.0" friction="0.0" />
@@ -486,6 +469,5 @@
             <origin rpy="0 ${-PI/2} ${PI/2}" xyz="0 0 0" />
             <axis xyz="0 0 1" />
-            <!--limit
-            effort and velocity picked arbitrarily check-->
+            <!-- Limit effort and velocity picked arbitrarily check -->
             <limit effort="100.0" lower="${-1.5*PI}" upper="${1.5*PI}" velocity="10" />
             <joint_properties damping="1.0" friction="0.0" />

Commit message: Added Mimic Joint limits and Fixed Mimic Joint types

File: ecm_description/urdf/xacros/ecm.xacro (robot description, xacro)
@@ -175,5 +175,5 @@
         </joint>
         <!-- Joint 5: Outer Pitch Joint 0: Link 3 to Link 5 -->
-        <joint name="${prefix}_outer_pitch_0" type="continuous">
+        <joint name="${prefix}_outer_pitch_0" type="revolute">
             <parent link="${prefix}_yaw_link" />
             <child link="${prefix}_pitch_link_1" />
@@ -181,8 +181,9 @@
             <axis xyz="0 0 1" />
             <joint_properties damping="1.0" friction="0.0" />
+            <limit effort="100.0" lower="${-PI/4}" upper="${PI*65/180}" velocity="10" />
             <mimic joint="${prefix}_outer_pitch" multiplier="1" />
         </joint>
         <!-- Joint 6: Outer Pitch Joint 1: Link 5 to Link 6 -->
-        <joint name="${prefix}_outer_pitch_1" type="continuous">
+        <joint name="${prefix}_outer_pitch_1" type="revolute">
             <parent link="${prefix}_pitch_link_1" />
             <child link="${prefix}_pitch_link_2" />
@@ -190,8 +191,9 @@
             <axis xyz="0 0 1" />
             <joint_properties damping="1.0" friction="0.0" />
+            <limit effort="100.0" upper="${PI/4}" lower="${-PI*65/180}" velocity="10" />
             <mimic joint="${prefix}_outer_pitch" multiplier="-1" />
         </joint>
         <!-- Joint 7: Outer Pitch Joint 2: Link 6 to Link 7 -->
-        <joint name="${prefix}_outer_pitch_2" type="continuous">
+        <joint name="${prefix}_outer_pitch_2" type="revolute">
             <parent link="${prefix}_pitch_link_2" />
             <child link="${prefix}_pitch_link_3" />
@@ -199,4 +201,5 @@
             <axis xyz="0 0 1" />
             <joint_properties damping="1.0" friction="0.0" />
+            <limit effort="100.0" lower="${-PI/4}" upper="${PI*65/180}" velocity="10" />
             <mimic joint="${prefix}_outer_pitch" multiplier="1" />
         </joint>
