Commit message: Minor Refactor

File: ecm_description/urdf/xacros/ecm.base.xacro (robot description, xacro)
@@ -4,6 +4,5 @@
     <xacro:include filename="$(find ecm_description)/urdf/xacros/common.xacro" />
     <!-- Macro for da Vinci Endoscope Camera Manipulator (ECM) Base -->
-    <xacro:macro name="ecm_base"
-        params="prefix parent_link xyz:='-0.612599 0.0 -0.101595' rpy:='0.0 0.0 0.0'">
+    <xacro:macro name="ecm_base" params="prefix parent_link xyz:='-0.612599 0.0 -0.101595' rpy:='0.0 0.0 0.0'">
         <!-- Link 0: Base Link -->
         <link name="${prefix}_base_link">

File: mtm_description/urdf/xacros/mtm.xacro (robot description, xacro)
@@ -7,5 +7,7 @@
     <!-- Macro for the da Vinci Master Console -->
     <xacro:macro name="master_console" params="prefix parent_link xyz rpy">
+        <!-- Link -1: Master Base Link -->
         <link name="${prefix}_master_base_link" />
+        <!-- Joint -1: Fixed to World: Parent Link to Link -1 -->
         <joint name="base_fixed" type="fixed">
             <parent link="${parent_link}" />
