Commit message: Refactor spacing in material names in ecmj.xacro

File: suj_description/urdf/xacros/Classic/ecmj.xacro (robot description, xacro)
@@ -12,5 +12,5 @@
                     <mesh filename="package://suj_description/meshes/Classic/suj_ecm_L0.stl" />
                 </geometry>
-                <material name="GrayBrown"/>
+                <material name="GrayBrown" />
             </visual>
             <collision>
@@ -28,5 +28,5 @@
                     <mesh filename="package://suj_description/meshes/Classic/suj_ecm_L1.stl" />
                 </geometry>
-                <material name="GrayBrown"/>
+                <material name="GrayBrown" />
             </visual>
             <collision>
@@ -44,5 +44,5 @@
                     <mesh filename="package://suj_description/meshes/Classic/suj_ecm_L2.stl" />
                 </geometry>
-                <material name="GrayBrown"/>
+                <material name="GrayBrown" />
             </visual>
             <collision>
@@ -60,5 +60,5 @@
                     <mesh filename="package://suj_description/meshes/Classic/suj_ecm_L3.stl" />
                 </geometry>
-                <material name="GrayBrown"/>
+                <material name="GrayBrown" />
             </visual>
             <collision>
@@ -77,5 +77,5 @@
             <child link="suj_ecm_L0" />
             <axis xyz="0 0 -1" />
-            <limit lower="-0.3798" upper="0.8425" effort="50" velocity ="50" />
+            <limit lower="-0.3798" upper="0.8425" effort="50" velocity="50" />
         </joint>
         <!-- Joint 8: ECM Joint 1: Link 8 to Link 9 -->
