Commit message: Refactor suj_description package to use separate xacro files for better organization

File: suj_description/urdf/suj.classic.urdf.xacro (robot description, xacro)
@@ -1,11 +1,14 @@
 <?xml version="1.0"?>
-<robot name="patient_cart" xmlns:xacro="http://www.ros.org/wiki/xacro">
+<robot name="suj_classic" xmlns:xacro="http://www.ros.org/wiki/xacro">
+    <!-- Mathematical Constants -->
     <xacro:property name="PI" value="3.1415926535897931" />
+    <!-- Macros -->
+    <xacro:include filename="$(find suj_description)/urdf/xacros/Classic/psm2j.xacro" />
+    <xacro:include filename="$(find suj_description)/urdf/xacros/Classic/ecmj.xacro" />
+    <xacro:include filename="$(find suj_description)/urdf/xacros/Classic/psm1j.xacro" />
+    <xacro:include filename="$(find suj_description)/urdf/xacros/Classic/psm3j.xacro" />
+    <!-- Link 0: World -->
     <link name="world" />
-    <joint name="fixed" type="fixed">
-        <origin xyz="0 0 0.167458" rpy="0 0 0" />
-        <parent link="world" />
-        <child link="base_link" />
-    </joint>
+    <!-- Link 1: Base Link -->
     <link name="base_link">
         <visual>
@@ -25,484 +28,29 @@
         </collision>
     </link>
-    <link name="suj_psm2_L0">
-        <visual>
-            <origin xyz="0 0 0" rpy="0 0 0" />
-            <geometry>
-                <mesh filename="package://suj_description/meshes/Classic/suj_psm2_L0.stl" />
-            </geometry>
-            <material name="">
-                <color rgba="0.792156862745098 0.819607843137255 0.933333333333333 1" />
-            </material>
-        </visual>
-        <collision>
-            <origin xyz="0 0 0" rpy="0 0 0" />
-            <geometry>
-                <mesh filename="package://suj_description/meshes/Classic/suj_psm2_L0.stl" />
-            </geometry>
-        </collision>
-    </link>
-    <joint name="SUJ_PSM2_J0" type="prismatic">
-        <origin xyz="0.1912 -0.101599999999999 0.761099999999999" rpy="-${PI} 0.0 ${PI}" />
-        <parent link="base_link" />
-        <child link="suj_psm2_L0" />
-        <axis xyz="0 0 -1" />
-        <limit
-            lower="-0.3798"
-            upper="0.8425"
-            effort="50"
-            velocity="50" />
+    <!-- Joint 0: Fixed: Link 0 to Link 1 -->
+    <joint name="fixed" type="fixed">
+        <origin xyz="0 0 0.167458" rpy="0 0 0" />
+        <parent link="world" />
+        <child link="base_link" />
     </joint>
-    <link name="suj_psm2_L1">
-        <visual>
-            <origin xyz="0 0 0" rpy="0 0 0" />
-            <geometry>
-                <mesh filename="package://suj_description/meshes/Classic/suj_psm2_L1.stl" />
-            </geometry>
-            <material name="">
-                <color rgba="0.792156862745098 0.819607843137255 0.933333333333333 1" />
-            </material>
-        </visual>
-        <collision>
-            <origin xyz="0 0 0" rpy="0 0 0" />
-            <geometry>
-                <mesh filename="package://suj_description/meshes/Classic/suj_psm2_L1.stl" />
-            </geometry>
-        </collision>
-    </link>
-    <joint name="SUJ_PSM2_J1" type="continuous">
-        <origin xyz="0 0 0" rpy="0 0 ${PI/2}" />
-        <parent link="suj_psm2_L0" />
-        <child link="suj_psm2_L1" />
-        <axis xyz="0 0 -1" />
-    </joint>
-    <link name="suj_psm2_L2">
-        <visual>
-            <origin xyz="0 0 0" rpy="0 0 0" />
-            <geometry>
-                <mesh filename="package://suj_description/meshes/Classic/suj_psm2_L2.stl" />
-            </geometry>
-            <material name="">
-                <color rgba="0.792156862745098 0.819607843137255 0.933333333333333 1" />
-            </material>
-        </visual>
-        <collision>
-            <origin xyz="0 0 0" rpy="0 0 0" />
-            <geometry>
-                <mesh filename="package://suj_description/meshes/Classic/suj_psm2_L2.stl" />
-            </geometry>
-        </collision>
-    </link>
-    <joint name="SUJ_PSM2_J2" type="continuous">
-        <origin xyz="0 0.4318 -0.17125" rpy="${PI} 0.0 ${PI/2}" />
-        <parent link="suj_psm2_L1" />
-        <child link="suj_psm2_L2" />
-        <axis xyz="0 0 1" />
-    </joint>
-    <link name="suj_psm2_L3">
-        <visual>
-            <origin xyz="0 0 0" rpy="0 0 0" />
-            <geometry>
-                <mesh filename="package://suj_description/meshes/Classic/suj_psm2_L3.stl" />
-            </geometry>
-            <material name="">
-                <color rgba="0.792156862745098 0.819607843137255 0.933333333333333 1" />
-            </material>
-        </visual>
-        <collision>
-            <origin xyz="0 0 0" rpy="0 0 0" />
-            <geometry>
-                <mesh filename="package://suj_description/meshes/Classic/suj_psm2_L3.stl" />
-            </geometry>
-        </collision>
-    </link>
-    <joint name="SUJ_PSM2_J3" type="continuous">
-        <origin xyz="0.4318 0 0" rpy="-${PI/2} 0 -${PI/2}" />
-        <parent link="suj_psm2_L2" />
-        <child link="suj_psm2_L3" />
-        <axis xyz="0 -1 0" />
-    </joint>
-    <link name="suj_psm2_L4">
-        <visual>
-            <origin xyz="0 0 0" rpy="0 0 0" />
-            <geometry>
-                <mesh filename="package://suj_description/meshes/Classic/suj_psm2_L4.stl" />
-            </geometry>
-            <material name="">
-                <color rgba="0.792156862745098 0.819607843137255 0.933333333333333 1" />
-            </material>
-        </visual>
-        <collision>
-            <origin xyz="0 0 0" rpy="0 0 0" />
-            <geometry>
-                <mesh filename="package://suj_description/meshes/Classic/suj_psm2_L4.stl" />
-            </geometry>
-        </collision>
-    </link>
-    <joint name="SUJ_PSM2_J4" type="continuous">
-        <origin xyz="0 0.0730499999999998 0.0609999999999997" rpy="${PI/2} 0.0 ${PI}" />
-        <parent link="suj_psm2_L3" />
-        <child link="suj_psm2_L4" />
-        <axis xyz="0 1 0" />
-    </joint>
-    <link name="PSM2_mounting_point" />
-    <joint name="PSM2_RCM" type="fixed">
-        <origin xyz="0.0 0.8343 -0.04984" rpy="0.0 ${PI} 0.0" />
-        <parent link="suj_psm2_L4" />
-        <child link="PSM2_mounting_point" />
-    </joint>
-    <link name="suj_ecm_L0">
-        <visual>
-            <origin xyz="0 0 0" rpy="0 0 0" />
-            <geometry>
-                <mesh filename="package://suj_description/meshes/Classic/suj_ecm_L0.stl" />
-            </geometry>
-            <material name="">
-                <color rgba="0.792156862745098 0.819607843137255 0.933333333333333 1" />
-            </material>
-        </visual>
-        <collision>
-            <origin xyz="0 0 0" rpy="0 0 0" />
-            <geometry>
-                <mesh filename="package://suj_description/meshes/Classic/suj_ecm_L0.stl" />
-            </geometry>
-        </collision>
-    </link>
-    <joint name="SUJ_ECM_J0" type="prismatic">
-        <origin xyz="0 0.0896 0.7611" rpy="${PI} 0 -${PI/2}" />
-        <parent link="base_link" />
-        <child link="suj_ecm_L0" />
-        <axis xyz="0 0 -1" />
-        <limit
-            lower="-0.3798"
-            upper="0.8425"
-            effort="50"
-            velocity="50" />
-    </joint>
-    <link name="suj_ecm_L1">
-        <visual>
-            <origin xyz="0 0 0" rpy="0 0 0" />
-            <geometry>
-                <mesh filename="package://suj_description/meshes/Classic/suj_ecm_L1.stl" />
-            </geometry>
-            <material name="">
-                <color rgba="0.792156862745098 0.819607843137255 0.933333333333333 1" />
-            </material>
-        </visual>
-        <collision>
-            <origin xyz="0 0 0" rpy="0 0 0" />
-            <geometry>
-                <mesh filename="package://suj_description/meshes/Classic/suj_ecm_L1.stl" />
-            </geometry>
-        </collision>
-    </link>
-    <joint name="SUJ_ECM_J1" type="continuous">
-        <origin xyz="0 0 0" rpy="${PI} 0 ${PI/2}" />
-        <parent link="suj_ecm_L0" />
-        <child link="suj_ecm_L1" />
-        <axis xyz="0 0 1" />
-    </joint>
-    <link name="suj_ecm_L2">
-        <visual>
-            <origin xyz="0 0 0" rpy="0 0 0" />
-            <geometry>
-                <mesh filename="package://suj_description/meshes/Classic/suj_ecm_L2.stl" />
-            </geometry>
-            <material name="">
-                <color rgba="0.792156862745098 0.819607843137255 0.933333333333333 1" />
-            </material>
-        </visual>
-        <collision>
-            <origin xyz="0 0 0" rpy="0 0 0" />
-            <geometry>
-                <mesh filename="package://suj_description/meshes/Classic/suj_ecm_L2.stl" />
-            </geometry>
-        </collision>
-    </link>
-    <joint name="SUJ_ECM_J2" type="continuous">
-        <origin xyz="0 -0.4318 0.17125" rpy="${PI} 0 -${PI/2}" />
-        <parent link="suj_ecm_L1" />
-        <child link="suj_ecm_L2" />
-        <axis xyz="0 0 -1" />
-    </joint>
-    <link name="suj_ecm_L3">
-        <visual>
-            <origin xyz="0 0 0" rpy="0 0 0" />
-            <geometry>
-                <mesh filename="package://suj_description/meshes/Classic/suj_ecm_L3.stl" />
-            </geometry>
-            <material name="">
-                <color rgba="0.792156862745098 0.819607843137255 0.933333333333333 1" />
-            </material>
-        </visual>
-        <collision>
-            <origin xyz="0 0 0" rpy="0 0 0" />
-            <geometry>
-                <mesh filename="package://suj_description/meshes/Classic/suj_ecm_L3.stl" />
-            </geometry>
-        </collision>
-    </link>
-    <joint name="SUJ_ECM_J3" type="continuous">
-        <origin xyz="0.4318 0.0 0.052" rpy="${PI/2} 0.0 0.0" />
-        <parent link="suj_ecm_L2" />
-        <child link="suj_ecm_L3" />
-        <axis xyz="0 -1 0" />
-    </joint>
-    <link name="ECM_mounting_point" />
-    <joint name="ECM_RCM" type="fixed">
-        <origin xyz="-0.45788 0.55053 0.0" rpy="${PI/2} ${PI} -${PI/4}" />
-        <parent link="suj_ecm_L3" />
-        <child link="ECM_mounting_point" />
-    </joint>
-    <link name="suj_psm1_L0">
-        <visual>
-            <origin xyz="0 0 0" rpy="0 0 0" />
-            <geometry>
-                <mesh filename="package://suj_description/meshes/Classic/suj_psm1_L0.stl" />
-            </geometry>
-            <material name="">
-                <color rgba="0.792156862745098 0.819607843137255 0.933333333333333 1" />
-            </material>
-        </visual>
-        <collision>
-            <origin xyz="0 0 0" rpy="0 0 0" />
-            <geometry>
-                <mesh filename="package://suj_description/meshes/Classic/suj_psm1_L0.stl" />
-            </geometry>
-        </collision>
-    </link>
-    <joint name="SUJ_PSM1_J0" type="prismatic">
-        <origin xyz="-0.191199999999999 -0.1016 0.761099999999999" rpy="${PI} 0 0" />
-        <parent link="base_link" />
-        <child link="suj_psm1_L0" />
-        <axis xyz="0 0 -1" />
-        <limit
-            lower="-0.3798"
-            upper="0.8425"
-            effort="50"
-            velocity="50" />
-    </joint>
-    <link name="suj_psm1_L1">
-        <visual>
-            <origin xyz="0 0 0" rpy="0 0 0" />
-            <geometry>
-                <mesh filename="package://suj_description/meshes/Classic/suj_psm1_L1.stl" />
-            </geometry>
-            <material name="">
-                <color rgba="0.792156862745098 0.819607843137255 0.933333333333333 1" />
-            </material>
-        </visual>
-        <collision>
-            <origin xyz="0 0 0" rpy="0 0 0" />
-            <geometry>
-                <mesh filename="package://suj_description/meshes/Classic/suj_psm1_L1.stl" />
-            </geometry>
-        </collision>
-    </link>
-    <joint name="SUJ_PSM1_J1" type="continuous">
-        <origin xyz="0 0 0" rpy="0 0 ${PI/2}" />
-        <parent link="suj_psm1_L0" />
-        <child link="suj_psm1_L1" />
-        <axis xyz="0 0 -1" />
-    </joint>
-    <link name="suj_psm1_L2">
-        <visual>
-            <origin xyz="0 0 0" rpy="0 0 0" />
-            <geometry>
-                <mesh filename="package://suj_description/meshes/Classic/suj_psm1_L2.stl" />
-            </geometry>
-            <material name="">
-                <color rgba="0.792156862745098 0.819607843137255 0.933333333333333 1" />
-            </material>
-        </visual>
-        <collision>
-            <origin xyz="0 0 0" rpy="0 0 0" />
-            <geometry>
-                <mesh filename="package://suj_description/meshes/Classic/suj_psm1_L2.stl" />
-            </geometry>
-        </collision>
-    </link>
-    <joint name="SUJ_PSM1_J2" type="continuous">
-        <origin xyz="0 0.4318 -0.171250000000001" rpy="${PI} 0 ${PI/2}" />
-        <parent link="suj_psm1_L1" />
-        <child link="suj_psm1_L2" />
-        <axis xyz="0 0 1" />
-    </joint>
-    <link name="suj_psm1_L3">
-        <visual>
-            <origin xyz="0 0 0" rpy="0 0 0" />
-            <geometry>
-                <mesh filename="package://suj_description/meshes/Classic/suj_psm1_L3.stl" />
-            </geometry>
-            <material name="">
-                <color rgba="0.792156862745098 0.819607843137255 0.933333333333333 1" />
-            </material>
-        </visual>
-        <collision>
-            <origin xyz="0 0 0" rpy="0 0 0" />
-            <geometry>
-                <mesh filename="package://suj_description/meshes/Classic/suj_psm1_L3.stl" />
-            </geometry>
-        </collision>
-    </link>
-    <joint name="SUJ_PSM1_J3" type="continuous">
-        <origin xyz="0.4318 0 0" rpy="${PI/2} 0 -${PI/2}" />
-        <parent link="suj_psm1_L2" />
-        <child link="suj_psm1_L3" />
-        <axis xyz="0 1 0" />
-    </joint>
-    <link name="suj_psm1_L4">
-        <visual>
-            <origin xyz="0 0 0" rpy="0 0 0" />
-            <geometry>
-                <mesh filename="package://suj_description/meshes/Classic/suj_psm1_L4.stl" />
-            </geometry>
-            <material name="">
-                <color rgba="0.792156862745098 0.819607843137255 0.933333333333333 1" />
-            </material>
-        </visual>
-        <collision>
-            <origin xyz="0 0 0" rpy="0 0 0" />
-            <geometry>
-                <mesh filename="package://suj_description/meshes/Classic/suj_psm1_L4.stl" />
-            </geometry>
-        </collision>
-    </link>
-    <joint name="SUJ_PSM1_J4" type="continuous">
-        <origin xyz="0 -0.0730499999999998 -0.0609999999999999" rpy="-${PI/2} 0 ${PI}" />
-        <parent link="suj_psm1_L3" />
-        <child link="suj_psm1_L4" />
-        <axis xyz="0 1 0" />
-    </joint>
-    <link name="PSM1_mounting_point" />
-    <joint name="PSM1_RCM" type="fixed">
-        <origin xyz="0.0 0.8343 -0.04984" rpy="0.0 ${PI} 0.0" />
-        <parent link="suj_psm1_L4" />
-        <child link="PSM1_mounting_point" />
-    </joint>
-    <link name="suj_psm3_L0">
-        <visual>
-            <origin xyz="0 0 0" rpy="0 0 0" />
-            <geometry>
-                <mesh filename="package://suj_description/meshes/Classic/suj_psm3_L0.stl" />
-            </geometry>
-            <material name="">
-                <color rgba="0.792156862745098 0.819607843137255 0.933333333333333 1" />
-            </material>
-        </visual>
-        <collision>
-            <origin xyz="0 0 0" rpy="0 0 0" />
-            <geometry>
-                <mesh filename="package://suj_description/meshes/Classic/suj_psm3_L0.stl" />
-            </geometry>
-        </collision>
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
Commit message: Added ROS2 Control for suj_desciption

File: suj_description/urdf/suj.classic.urdf.xacro (robot description, xacro)
@@ -8,4 +8,6 @@
     <xacro:include filename="$(find suj_description)/urdf/xacros/Classic/psm1j.xacro" />
     <xacro:include filename="$(find suj_description)/urdf/xacros/Classic/psm3j.xacro" />
+    <xacro:include filename="$(find suj_description)/urdf/ros2_control/ecmj.ros2_control.xacro" />
+    <xacro:include filename="$(find suj_description)/urdf/ros2_control/psmj.ros2_control.xacro" />
     <!-- Link 0: World -->
     <link name="world" />
@@ -38,10 +40,10 @@
         parent_link="base_link"
         xyz="0.1912 -0.101599999999999 0.761099999999999"
-        rpy="-${PI} 0.0 ${PI}"/>
+        rpy="-${PI} 0.0 ${PI}" />
     <!-- ECM -->
     <xacro:ecm_j
         parent_link="base_link"
         xyz="0 0.0896 0.7611"
-        rpy="${PI} 0 -${PI/2}"/>
+        rpy="${PI} 0 -${PI/2}" />
     <!-- PSM 1 -->
     <xacro:psm1_j
@@ -53,4 +55,7 @@
         parent_link="base_link"
         xyz="0 0.0895999999999999 0.3813"
-        rpy="${PI} 0 -${PI/2}"/>
+        rpy="${PI} 0 -${PI/2}" />
+    <!-- ROS2 Control -->
+    <xacro:ecmj_ros2_control />
+    <xacro:psmj_ros2_control />
 </robot>

File: suj_description/urdf/suj.si.urdf.xacro (robot description, xacro)
@@ -7,4 +7,6 @@
     <xacro:include filename="$(find suj_description)/urdf/xacros/Si/psm3j.xacro" />
     <xacro:include filename="$(find suj_description)/urdf/xacros/Si/ecmj.xacro" />
+    <xacro:include filename="$(find suj_description)/urdf/ros2_control/ecmj.ros2_control.xacro" />
+    <xacro:include filename="$(find suj_description)/urdf/ros2_control/psmj.ros2_control.xacro" />
     <!-- Link 0: World -->
     <link name="world" />
@@ -14,5 +16,6 @@
             <origin xyz="-1.969E-09 2.3996E-09 0.80012" rpy="0 0 0" />
             <mass value="71.07" />
-            <inertia ixx="16.038" ixy="-5.7683E-10" ixz="8.3859E-08" iyy="16.017" iyz="-1.008E-07" izz="0.56653" />
+            <inertia ixx="16.038" ixy="-5.7683E-10" ixz="8.3859E-08" iyy="16.017" iyz="-1.008E-07"
+                izz="0.56653" />
         </inertial>
         <visual>
@@ -60,3 +63,6 @@
         xyz="0.223 0 0.528"
         rpy="0 0 0" />
+    <!-- ROS2 Control -->
+    <xacro:ecmj_ros2_control />
+    <xacro:psmj_ros2_control />
 </robot>
