Commit message: Added ROS2 Control for psm_desciption

File: psm_description/urdf/both_psms.classic.urdf.xacro (robot description, xacro)
@@ -3,4 +3,5 @@
     <!-- Macros -->
     <xacro:include filename="$(find psm_description)/urdf/xacros/Classic/psm.base.xacro" />
+    <xacro:include filename="$(find psm_description)/urdf/ros2_control/Classic/psm.base.ros2_control.xacro" />
     <!-- Parent Link -->
     <link name="world" />
@@ -17,11 +18,14 @@
     <!-- PSM Base 1 -->
     <xacro:psm_base
-        prefix="one_"
+        prefix="one"
         parent_link="camera"
         xyz="-0.25 0.0 0.5" rpy="0.0 0.0 ${PI}" />
     <!-- PSM Base 2 -->
     <xacro:psm_base
-        prefix="two_"
+        prefix="two"
         parent_link="camera"
         xyz="0.25 0.0 0.5" rpy="0.0 0.0 ${PI}" />
+    <!-- ROS2 Control -->
+    <xacro:psm_base_ros2_control prefix="one" />
+    <xacro:psm_base_ros2_control prefix="two" />
 </robot>

File: psm_description/urdf/psm.classic.urdf.xacro (robot description, xacro)
@@ -3,6 +3,7 @@
     <!-- Tool Arguments -->
     <!-- Select tool_name from blade, caudier_blade, caudier, sca_blade, sca, snake -->
-    <xacro:property name="tool_name" default="sca" />
-    <xacro:property name="prefix" default="" />
+    <xacro:arg name="tool" default="sca" />
+    <xacro:property name="tool_name" default="'$(arg tool)'" />
+    <xacro:property name="prefix" default="PSM" />
     <xacro:property name="parent_link" default="world" />
     <!-- Tool Origin Arguments: for Caudier tool -->
@@ -19,4 +20,6 @@
     <xacro:include filename="$(find psm_description)/urdf/xacros/Classic/psm.base.xacro" />
     <xacro:include filename="$(find psm_description)/urdf/xacros/Classic/psm.tool.xacro" />
+    <xacro:include filename="$(find psm_description)/urdf/ros2_control/Classic/psm.base.ros2_control.xacro" />
+    <xacro:include filename="$(find psm_description)/urdf/ros2_control/Classic/psm.tool.ros2_control.xacro" />
     <!-- Parent Link -->
     <link name="${parent_link}" />
@@ -30,3 +33,6 @@
         prefix="${prefix}"
         parent_link="${prefix}_tool_wrist_shaft_link" />
+    <!-- ROS2 Control -->
+    <xacro:psm_base_ros2_control prefix="${prefix}" />
+    <xacro:psm_tool_ros2_control tool_name="${tool_name}" prefix="${prefix}" />
 </robot>

File: psm_description/urdf/psm.si.urdf.xacro (robot description, xacro)
@@ -4,8 +4,11 @@
     <xacro:include filename="$(find psm_description)/urdf/xacros/Si/psm.base.xacro" />
     <xacro:include filename="$(find psm_description)/urdf/xacros/Si/psm.tool.xacro" />
+    <xacro:include filename="$(find psm_description)/urdf/ros2_control/Si/psm.base.ros2_control.xacro" />
+    <xacro:include filename="$(find psm_description)/urdf/ros2_control/Si/psm.tool.ros2_control.xacro" />
     <!-- Tool Arguments -->
     <!-- Select tool_name from P420006, SF826001 -->
-    <xacro:property name="tool_name" default="P420006" />
-    <xacro:property name="prefix" default="" />
+    <xacro:arg name="tool" default="P420006" />
+    <xacro:property name="tool_name" default="'$(arg tool)'" />
+    <xacro:property name="prefix" default="PSM" />
     <xacro:property name="parent_link" default="world" />
     <xacro:property name="xyz" default="0.0 0.0 0.0" />
@@ -23,3 +26,6 @@
         parent_link="${prefix}_tool_parent"
         xyz="${xyz}" rpy="${rpy}" />
+    <!-- ROS2 Control -->
+    <xacro:psm_base_ros2_control prefix="${prefix}" />
+    <xacro:psm_tool_ros2_control tool_name="${tool_name}" prefix="${prefix}" />
 </robot>
