Commit message: Added ROS2 Control for patient_cart_desciption

File: patient_cart_description/urdf/patient_cart.classic.urdf.xacro (robot description, xacro)
@@ -11,6 +11,13 @@
     <xacro:include filename="$(find psm_description)/urdf/xacros/Classic/psm.tool.xacro" />
     <xacro:include filename="$(find ecm_description)/urdf/xacros/ecm.base.xacro" />
+    <!-- ROS2 Macros -->
+    <xacro:include filename="$(find suj_description)/urdf/ros2_control/ecmj.ros2_control.xacro" />
+    <xacro:include filename="$(find suj_description)/urdf/ros2_control/psmj.ros2_control.xacro" />
+    <xacro:include filename="$(find psm_description)/urdf/ros2_control/Classic/psm.base.ros2_control.xacro" />
+    <xacro:include filename="$(find psm_description)/urdf/ros2_control/Classic/psm.tool.ros2_control.xacro" />
+    <xacro:include filename="$(find ecm_description)/urdf/ros2_control/ecm.base.ros2_control.xacro" />
     <!-- Link 0: World -->
-    <link name="world" />
+    <link
+        name="world" />
     <!-- Link 1: Base Link -->
     <link name="base_link">
@@ -90,3 +97,18 @@
         prefix="PSM3"
         parent_link="PSM3_tool_wrist_shaft_link" />
+    <!-- ROS2 Control -->
+    <ros2_control name="patient_cart_classic_ros2_control" type="system">
+        <hardware>
+            <plugin>fake_components/GenericSystem</plugin>
+        </hardware>
+        <xacro:ecm_base_ros2_control prefix="ECM" />
+        <xacro:ecmj_ros2_control />
+        <xacro:psmj_ros2_control />
+        <xacro:psm_base_ros2_control prefix="PSM1" />
+        <xacro:psm_tool_ros2_control tool_name="sca" prefix="PSM1" />
+        <xacro:psm_base_ros2_control prefix="PSM2" />
+        <xacro:psm_tool_ros2_control tool_name="caudier" prefix="PSM2" />
+        <xacro:psm_base_ros2_control prefix="PSM3" />
+        <xacro:psm_tool_ros2_control tool_name="caudier" prefix="PSM3" />
+    </ros2_control>
 </robot>

File: patient_cart_description/urdf/patient_cart.si.urdf.xacro (robot description, xacro)
@@ -10,4 +10,10 @@
     <xacro:include filename="$(find psm_description)/urdf/xacros/Si/psm.tool.xacro" />
     <xacro:include filename="$(find ecm_description)/urdf/xacros/ecm.base.xacro" />
+    <!-- ROS2 Macros -->
+    <xacro:include filename="$(find suj_description)/urdf/ros2_control/ecmj.ros2_control.xacro" />
+    <xacro:include filename="$(find suj_description)/urdf/ros2_control/psmj.ros2_control.xacro" />
+    <xacro:include filename="$(find psm_description)/urdf/ros2_control/Si/psm.base.ros2_control.xacro" />
+    <xacro:include filename="$(find psm_description)/urdf/ros2_control/Si/psm.tool.ros2_control.xacro" />
+    <xacro:include filename="$(find ecm_description)/urdf/ros2_control/ecm.base.ros2_control.xacro" />
     <!-- Link 0: World -->
     <link name="world" />
@@ -70,6 +76,5 @@
         xyz="0.0 0.0 0.0" rpy="0.0 0.0 0.0" />
     <!-- ECM Link -->
-    <xacro:psm_tool
-        tool_name="SF826001"
+    <xacro:ecm_base
         prefix="ECM"
         parent_link="ECM_mounting_point"
@@ -95,3 +100,18 @@
         parent_link="PSM3_tool_parent"
         xyz="0.0 0.0 0.0" rpy="0.0 0.0 0.0" />
+    <!-- ROS2 Control -->
+    <ros2_control name="patient_cart_si_ros2_control" type="system">
+        <hardware>
+            <plugin>fake_components/GenericSystem</plugin>
+        </hardware>
+        <xacro:ecmj_ros2_control />
+        <xacro:psmj_ros2_control />
+        <xacro:ecm_base_ros2_control prefix="ECM" />
+        <xacro:psm_base_ros2_control prefix="PSM1" />
+        <xacro:psm_tool_ros2_control tool_name="P420006" prefix="PSM1" />
+        <xacro:psm_base_ros2_control prefix="PSM2" />
+        <xacro:psm_tool_ros2_control tool_name="P420006" prefix="PSM2" />
+        <xacro:psm_base_ros2_control prefix="PSM3" />
+        <xacro:psm_tool_ros2_control tool_name="P420006" prefix="PSM3" />
+    </ros2_control>
 </robot>
