Commit message: Added comments for ROS2 control macros

File: davinci_core_description/urdf/ros2_control/daVinci.arm.ros2_control.xacro (robot description, xacro)
@@ -1,5 +1,7 @@
 <?xml version="1.0"?>
 <robot xmlns:xacro="http://www.ros.org/wiki/xacro">
+    <!-- ROS2 Control Macro for the daVinci arm -->
     <xacro:macro name="davinci_core_ros2_control" params="arm_name">
+        <!-- Command Joint 0 -->
         <joint name="${arm_name}_outer_yaw_joint">
             <command_interface name="position" />
@@ -7,4 +9,5 @@
             <state_interface name="velocity" />
         </joint>
+        <!-- Command Joint 1 -->
         <joint name="${arm_name}_outer_pitch_base_joint">
             <command_interface name="position" />
@@ -12,4 +15,5 @@
             <state_interface name="velocity" />
         </joint>
+        <!-- Command Joint 2 -->
         <joint name="${arm_name}_outer_pitch_front_joint">
             <command_interface name="position" />
@@ -17,4 +21,5 @@
             <state_interface name="velocity" />
         </joint>
+        <!-- Command Joint 3 -->
         <joint name="${arm_name}_outer_pitch_bottom_joint">
             <command_interface name="position" />
@@ -22,4 +27,5 @@
             <state_interface name="velocity" />
         </joint>
+        <!-- Command Joint 4 -->
         <joint name="${arm_name}_outer_pitch_top_joint">
             <command_interface name="position" />
@@ -27,4 +33,5 @@
             <state_interface name="velocity" />
         </joint>
+        <!-- Command Joint 5 -->
         <joint name="${arm_name}_outer_insertion_joint">
             <command_interface name="position" />
@@ -32,4 +39,5 @@
             <state_interface name="velocity" />
         </joint>
+        <!-- Command Joint 6 -->
         <joint name="${arm_name}_tool_insertion_joint">
             <command_interface name="position" />

File: ecm_description/urdf/ros2_control/ecm.base.ros2_control.xacro (robot description, xacro)
@@ -1,6 +1,7 @@
 <?xml version="1.0"?>
 <robot xmlns:xacro="http://www.ros.org/wiki/xacro">
+    <!-- ROS2 Control Macro for the ECM base -->
     <xacro:macro name="ecm_base_ros2_control" params="prefix">
-        <!-- Define the joints and their interfaces -->
+        <!-- Command Joint 0 -->
         <joint name="${prefix}_yaw">
             <command_interface name="position" />
@@ -8,4 +9,5 @@
             <state_interface name="velocity" />
         </joint>
+        <!-- Command Joint 1 -->
         <joint name="${prefix}_pitch">
             <command_interface name="position" />
@@ -13,4 +15,5 @@
             <state_interface name="velocity" />
         </joint>
+        <!-- Command Joint 2 -->
         <joint name="${prefix}_insertion">
             <command_interface name="position" />
@@ -18,4 +21,5 @@
             <state_interface name="velocity" />
         </joint>
+        <!-- Command Joint 3 -->
         <joint name="${prefix}_roll">
             <command_interface name="position" />
@@ -23,17 +27,20 @@
             <state_interface name="velocity" />
         </joint>
-        <!-- Mimic Joints -->
+        <!-- Mimic Joint 0: Command Joint 1 -->
         <joint name="${prefix}_pitch_bottom">
             <state_interface name="position" />
             <state_interface name="velocity" />
         </joint>
+        <!-- Mimic Joint 1: Command Joint 1 -->
         <joint name="${prefix}_pitch_end">
             <state_interface name="position" />
             <state_interface name="velocity" />
         </joint>
+        <!-- Mimic Joint 2: Command Joint 1 -->
         <joint name="${prefix}_pitch_top">
             <state_interface name="position" />
             <state_interface name="velocity" />
         </joint>
+        <!-- Mimic Joint 3: Command Joint 1 -->
         <joint name="${prefix}_pitch_back">
             <state_interface name="position" />

File: ecm_description/urdf/ros2_control/ecm.ros2_control.xacro (robot description, xacro)
@@ -1,5 +1,7 @@
 <?xml version="1.0"?>
 <robot xmlns:xacro="http://www.ros.org/wiki/xacro">
+    <!-- ROS2 Control Macro for the ECM -->
     <xacro:macro name="ecm_ros2_control" params="prefix">
+        <!-- Command Joint 0 -->
         <joint name="${prefix}_outer_yaw">
             <command_interface name="position" />
@@ -7,4 +9,5 @@
             <state_interface name="velocity" />
         </joint>
+        <!-- Command Joint 1 -->
         <joint name="${prefix}_outer_pitch">
             <command_interface name="position" />
@@ -12,23 +15,27 @@
             <state_interface name="velocity" />
         </joint>
-        <joint name="${prefix}_insertion" type="prismatic">
+        <!-- Command Joint 2 -->
+        <joint name="${prefix}_insertion">
             <command_interface name="position" />
             <state_interface name="position" />
             <state_interface name="velocity" />
         </joint>
-        <joint name="${prefix}_outer_roll" type="revolute">
+        <!-- Command Joint 3 -->
+        <joint name="${prefix}_outer_roll">
             <command_interface name="position" />
             <state_interface name="position" />
             <state_interface name="velocity" />
         </joint>
-        <!-- Mimic Joints -->
+        <!-- Mimic Joint 0: Command Joint 1 -->
         <joint name="${prefix}_outer_pitch_0">
             <state_interface name="position" />
             <state_interface name="velocity" />
         </joint>
+        <!-- Mimic Joint 1: Command Joint 1 -->
         <joint name="${prefix}_outer_pitch_1">
             <state_interface name="position" />
             <state_interface name="velocity" />
         </joint>
+        <!-- Mimic Joint 2: Command Joint 1 -->
         <joint name="${prefix}_outer_pitch_2">
             <state_interface name="position" />

File: mtm_description/urdf/ros2_control/mtm.ros2_control.xacro (robot description, xacro)
@@ -1,7 +1,8 @@
 <?xml version="1.0"?>
 <robot xmlns:xacro="http://www.ros.org/wiki/xacro">
+    <!-- ROS2 Control Macro for the MTM -->
     <xacro:macro name="mtm_ros2_control" params="prefix">
-        <!-- Define the joints and their interfaces -->
-        <!-- xacro:macro name="mtm" -->
+        <!-- ========================= xacro:macro name="mtm" ========================= -->
+        <!-- Command Joint 0 -->
         <joint name="${prefix}_outer_yaw">
             <command_interface name="position" />
@@ -9,4 +10,5 @@
             <state_interface name="velocity" />
         </joint>
+        <!-- Command Joint 1 -->
         <joint name="${prefix}_shoulder_pitch">
             <command_interface name="position" />
@@ -14,4 +16,5 @@
             <state_interface name="velocity" />
         </joint>
+        <!-- Command Joint 2 -->
         <joint name="${prefix}_elbow_pitch">
             <command_interface name="position" />
@@ -19,5 +22,6 @@
             <state_interface name="velocity" />
         </joint>
-        <!-- xacro:macro name="mtm_platform_<`left` or `right`>" -->
+        <!-- ========================= xacro:macro name="mtm_platform_<`left` or `right`>" ========================= -->
+        <!-- Command Joint 3 -->
         <joint name="${prefix}_wrist_platform">
             <command_interface name="position" />
@@ -25,4 +29,5 @@
             <state_interface name="velocity" />
         </joint>
+        <!-- Command Joint 4 -->
         <joint name="${prefix}_wrist_pitch">
             <command_interface name="position" />
@@ -30,4 +35,5 @@
             <state_interface name="velocity" />
         </joint>
+        <!-- Command Joint 5 -->
         <joint name="${prefix}_wrist_yaw">
             <command_interface name="position" />
@@ -35,4 +41,5 @@
             <state_interface name="velocity" />
         </joint>
+        <!-- Command Joint 6 -->
         <joint name="${prefix}_wrist_roll">
             <command_interface name="position" />
@@ -40,5 +47,5 @@
             <state_interface name="velocity" />
         </joint>
-        <!-- Mimic Joints -->
+        <!-- Mimic Joint 0: Command Joint 1 -->
         <joint name="${prefix}_shoulder_pitch_parallel">
             <state_interface name="position" />

File: suj_description/urdf/ros2_control/ecmj.ros2_control.xacro (robot description, xacro)
@@ -1,5 +1,7 @@
 <?xml version="1.0"?>
 <robot xmlns:xacro="http://www.ros.org/wiki/xacro">
+    <!-- ROS2 Control Macro for the ECM Joints -->
     <xacro:macro name="ecmj_ros2_control">
+        <!-- Command Joint 0 -->
         <joint name="SUJ_ECM_J0">
             <command_interface name="position" />
@@ -7,4 +9,5 @@
             <state_interface name="velocity" />
         </joint>
+        <!-- Command Joint 1 -->
         <joint name="SUJ_ECM_J1">
             <command_interface name="position" />
@@ -12,4 +15,5 @@
             <state_interface name="velocity" />
         </joint>
+        <!-- Command Joint 2 -->
         <joint name="SUJ_ECM_J2">
             <command_interface name="position" />
@@ -17,4 +21,5 @@
             <state_interface name="velocity" />
         </joint>
+        <!-- Command Joint 3 -->
         <joint name="SUJ_ECM_J3">
             <command_interface name="position" />

File: suj_description/urdf/ros2_control/psmj.ros2_control.xacro (robot description, xacro)
@@ -1,5 +1,7 @@
 <?xml version="1.0"?>
 <robot xmlns:xacro="http://www.ros.org/wiki/xacro">
+    <!-- ROS2 Control Macro for the PSM Joints -->
     <xacro:macro name="psmj_ros2_control" params="prefix">
+        <!-- Command Joint 0 -->
         <joint name="SUJ_PSM${prefix}_J0">
             <command_interface name="position" />
@@ -7,4 +9,5 @@
             <state_interface name="velocity" />
         </joint>
+        <!-- Command Joint 1 -->
         <joint name="SUJ_PSM${prefix}_J1">
             <command_interface name="position" />
@@ -12,4 +15,5 @@
             <state_interface name="velocity" />
         </joint>
+        <!-- Command Joint 2 -->
         <joint name="SUJ_PSM${prefix}_J2">
             <command_interface name="position" />
@@ -17,4 +21,5 @@
             <state_interface name="velocity" />
         </joint>
+        <!-- Command Joint 3 -->
         <joint name="SUJ_PSM${prefix}_J3">
             <command_interface name="position" />
@@ -22,4 +27,5 @@
             <state_interface name="velocity" />
         </joint>
+        <!-- Command Joint 4 -->
         <joint name="SUJ_PSM${prefix}_J4">
             <command_interface name="position" />
