Commit message: Minor Refactor

File: psm_description/urdf/xacros/Si/psm.base.xacro (robot description, xacro)
@@ -5,5 +5,5 @@
     <!-- Macro for da Vinci Si PSM Base -->
     <xacro:macro name="psm_base" params="prefix parent_link xyz:='0.0 0.0 0.0' rpy:='0.0 0.0 0.0'">
-        <!-- Link 0: -->
+        <!-- Link 0: Link 0 -->
         <link name="${prefix}_link_0">
             <inertial>
@@ -28,5 +28,5 @@
             </collision>
         </link>
-        <!-- Link 1: -->
+        <!-- Link 1: Link 1 -->
         <link name="${prefix}_link_1">
             <inertial>
@@ -40,5 +40,5 @@
                     <mesh filename="package://psm_description/meshes/Si/link_1.stl" />
                 </geometry>
-                <material name="Lavender"/>
+                <material name="Lavender" />
             </visual>
             <collision>
@@ -49,5 +49,5 @@
             </collision>
         </link>
-        <!-- Link 2: -->
+        <!-- Link 2: Link 2 -->
         <link name="${prefix}_link_2">
             <inertial>
@@ -61,5 +61,5 @@
                     <mesh filename="package://psm_description/meshes/Si/link_2.stl" />
                 </geometry>
-                <material name="Lavender"/>
+                <material name="Lavender" />
             </visual>
             <collision>
@@ -70,5 +70,5 @@
             </collision>
         </link>
-        <!-- Link 3: -->
+        <!-- Link 3: Link 3 -->
         <link name="${prefix}_link_3">
             <inertial>
@@ -82,5 +82,5 @@
                     <mesh filename="package://psm_description/meshes/Si/link_3.stl" />
                 </geometry>
-                <material name="Lavender"/>
+                <material name="Lavender" />
             </visual>
             <collision>
@@ -91,5 +91,5 @@
             </collision>
         </link>
-        <!-- Link 4: -->
+        <!-- Link 4: Link 4 -->
         <link name="${prefix}_link_4">
             <inertial>
@@ -103,5 +103,5 @@
                     <mesh filename="package://psm_description/meshes/Si/link_4.stl" />
                 </geometry>
-                <material name="Lavender"/>
+                <material name="Lavender" />
             </visual>
             <collision>
@@ -112,5 +112,5 @@
             </collision>
         </link>
-        <!-- Link 5: -->
+        <!-- Link 5: Tool Parent Link -->
         <link name="${prefix}_tool_parent" />
         <!-- Link 6: RCM Link -->
